Commit message: Add more colors

File: sd_simulation/description/colors.xacro (robot description, xacro)
@@ -2,17 +2,26 @@
 <robot xmlns:xacro="http://www.ros.org/wiki/xacro" name="colors">
     <material name="white">
-        <color rgba="1 1 1 1" />
+        <color rgba="1.0 1.0 1.0 1.0"/>
     </material>
     <material name="red">
-        <color rgba="1 0 0 1"/>
+        <color rgba="0.8 0.0 0.0 1.0"/>
     </material>
     <material name="orange">
-        <color rgba="1 0.3 0.1 1"/>
+        <color rgba="${255/255} ${108/255} ${10/255} 1.0"/>
     </material>
     <material name="blue">
-        <color rgba="0.2 0.2 1 1"/>
+        <color rgba="0.0 0.0 0.8 1.0"/>
+    </material>
+    <material name="green">
+        <color rgba="0.0 0.8 0.0 1.0"/>
+    </material>
+    <material name="grey">
+        <color rgba="0.2 0.2 0.2 1.0"/>
+    </material>
+    <material name="brown">
+        <color rgba="${222/255} ${207/255} ${195/255} 1.0"/>
     </material>
     <material name="black">
-        <color rgba="0 0 0 1"/>
+        <color rgba="0.0 0.0 0.0 1.0"/>
     </material>
 </robot>
