Commit message: Modify body-wheel joints

File: sd_simulation/description/body.xacro (robot description, xacro)
@@ -32,5 +32,5 @@
     <!-- LEFT WHEEL LINK -->
     <joint name="left_wheel_joint" type="continuous">
-        <parent link="base_link"/>
+        <parent link="chassis"/>
         <child link="left_wheel"/>
         <origin xyz="0 0.175 0" rpy="-${pi/2} 0 0" />
@@ -58,5 +58,5 @@
     <!-- RIGHT WHEEL LINK -->
     <joint name="right_wheel_joint" type="continuous">
-        <parent link="base_link"/>
+        <parent link="chassis"/>
         <child link="right_wheel"/>
         <origin xyz="0 -0.175 0" rpy="${pi/2} 0 0" />

Commit message: Change parent links to base_link

File: sd_simulation/description/body.xacro (robot description, xacro)
@@ -32,5 +32,5 @@
     <!-- LEFT WHEEL LINK -->
     <joint name="left_wheel_joint" type="continuous">
-        <parent link="chassis"/>
+        <parent link="base_link"/>
         <child link="left_wheel"/>
         <origin xyz="0 0.175 0" rpy="-${pi/2} 0 0" />
@@ -58,5 +58,5 @@
     <!-- RIGHT WHEEL LINK -->
     <joint name="right_wheel_joint" type="continuous">
-        <parent link="chassis"/>
+        <parent link="base_link"/>
         <child link="right_wheel"/>
         <origin xyz="0 -0.175 0" rpy="${pi/2} 0 0" />
@@ -84,5 +84,5 @@
     <!-- CASTER WHEEL LINK -->
     <joint name="caster_wheel_joint" type="fixed">
-        <parent link="chassis"/>
+        <parent link="base_link"/>
         <child link="caster_wheel"/>
         <origin xyz="0.24 0 0"/>

File: sd_simulation/description/lidar.xacro (robot description, xacro)
@@ -2,5 +2,5 @@
 <robot xmlns:xacro="http://www.ros.org/wiki/xacro" >
     <joint name="laser_joint" type="fixed">
-        <parent link="chassis"/>
+        <parent link="base_link"/>
         <child link="laser_frame"/>
         <origin xyz="0.1 0 0.175" rpy="0 0 0"/>

Commit message: Avoid using reserved link name 'chassis'

File: sd_simulation/description/body.xacro (robot description, xacro)
@@ -3,11 +3,11 @@
     <!-- BASE LINK -->
     <link name="base_link"/>
-    <!-- CHASSIS LINK -->
-    <joint name="chassis_joint" type="fixed">
+    <!-- BODY LINK -->
+    <joint name="body_joint" type="fixed">
         <parent link="base_link"/>
-        <child link="chassis"/>
+        <child link="body"/>
         <origin xyz="-0.1 0 0"/>
     </joint>
-    <link name="chassis">
+    <link name="body">
         <visual>
             <origin xyz="0.15 0 0.075"/>
@@ -27,5 +27,5 @@
         </xacro:inertial_box>
     </link>
-    <gazebo reference="chassis">
+    <gazebo reference="body">
         <material>Gazebo/White</material>
     </gazebo>
@@ -84,5 +84,5 @@
     <!-- CASTER WHEEL LINK -->
     <joint name="caster_wheel_joint" type="fixed">
-        <parent link="base_link"/>
+        <parent link="body"/>
         <child link="caster_wheel"/>
         <origin xyz="0.24 0 0"/>

File: sd_simulation/description/camera.xacro (robot description, xacro)
@@ -12,5 +12,5 @@
         <parent link="base_link"/>
         <child link="front_cam_link"/>
-        <origin xyz="0.3 0 0.1" rpy="0 0 0"/>
+        <origin xyz="0.2 0 0.1" rpy="0 0 0"/>
     </joint>
     <!-- We need to add the “dummy” link called camera_link_optical,

Commit message: Change wheels color

File: sd_simulation/description/body.xacro (robot description, xacro)
@@ -15,4 +15,5 @@
                 <box size="0.3 0.3 0.15"/>
             </geometry>
+            <!-- Color for RVIZ -->
             <material name="white"/>
         </visual>
@@ -27,4 +28,5 @@
         </xacro:inertial_box>
     </link>
+    <!-- Color for Gazebo -->
     <gazebo reference="body">
         <material>Gazebo/White</material>
@@ -42,5 +44,5 @@
                 <cylinder radius="0.05" length="0.04"/>
             </geometry>
-            <material name="blue"/>
+            <material name="yellow"/>
         </visual>
         <collision>
@@ -54,5 +56,5 @@
     </link>
     <gazebo reference="left_wheel">
-        <material>Gazebo/Blue</material>
+        <material>Gazebo/Wood</material>
     </gazebo>
     <!-- RIGHT WHEEL LINK -->
@@ -68,5 +70,5 @@
                 <cylinder radius="0.05" length="0.04"/>
             </geometry>
-            <material name="blue"/>
+            <material name="yellow"/>
         </visual>
         <collision>
@@ -80,5 +82,5 @@
     </link>
     <gazebo reference="right_wheel">
-        <material>Gazebo/Blue</material>
+        <material>Gazebo/Wood</material>
     </gazebo>
     <!-- CASTER WHEEL LINK -->

File: sd_simulation/description/colors.xacro (robot description, xacro)
@@ -9,4 +9,7 @@
     <material name="orange">
         <color rgba="${255/255} ${108/255} ${10/255} 1.0"/>
+    </material>
+    <material name="yellow">
+        <color rgba="0.8 0.8 0.0 1.0"/>
     </material>
     <material name="blue">

Commit message: Change robotBaseFrame to base_link; chassis was not a reserved link name

File: sd_simulation/description/body.xacro (robot description, xacro)
@@ -3,11 +3,11 @@
     <!-- BASE LINK -->
     <link name="base_link"/>
-    <!-- BODY LINK -->
-    <joint name="body_joint" type="fixed">
+    <!-- CHASSIS LINK -->
+    <joint name="chassis_joint" type="fixed">
         <parent link="base_link"/>
-        <child link="body"/>
+        <child link="chassis"/>
         <origin xyz="-0.1 0 0"/>
     </joint>
-    <link name="body">
+    <link name="chassis">
         <visual>
             <origin xyz="0.15 0 0.075"/>
@@ -29,5 +29,5 @@
     </link>
     <!-- Color for Gazebo -->
-    <gazebo reference="body">
+    <gazebo reference="chassis">
         <material>Gazebo/White</material>
     </gazebo>
@@ -86,5 +86,5 @@
     <!-- CASTER WHEEL LINK -->
     <joint name="caster_wheel_joint" type="fixed">
-        <parent link="body"/>
+        <parent link="chassis"/>
         <child link="caster_wheel"/>
         <origin xyz="0.24 0 0"/>

File: sd_simulation/description/gazebo_control.xacro (robot description, xacro)
@@ -16,5 +16,5 @@
             <!-- Output -->
             <odometryFrame>odom</odometryFrame>
-            <robotBaseFrame>chassis</robotBaseFrame>
+            <robotBaseFrame>base_link</robotBaseFrame>
             <!-- Others -->
             <rosDebugLevel>Debug</rosDebugLevel>

Commit message: Increase size of wheels

File: sd_simulation/description/body.xacro (robot description, xacro)
@@ -42,5 +42,5 @@
         <visual>
             <geometry>
-                <cylinder radius="0.05" length="0.04"/>
+                <cylinder radius="0.08" length="0.04"/>
             </geometry>
             <material name="yellow"/>
@@ -48,8 +48,8 @@
         <collision>
             <geometry>
-                <sphere radius="0.05"/>
+                <sphere radius="0.08"/>
             </geometry>
         </collision>
-        <xacro:inertial_cylinder mass="0.1" length="0.04" radius="0.05">
+        <xacro:inertial_cylinder mass="0.1" length="0.04" radius="0.08">
             <origin xyz="0 0 0" rpy="0 0 0"/>
         </xacro:inertial_cylinder>
@@ -68,5 +68,5 @@
         <visual>
             <geometry>
-                <cylinder radius="0.05" length="0.04"/>
+                <cylinder radius="0.08" length="0.04"/>
             </geometry>
             <material name="yellow"/>
@@ -74,8 +74,8 @@
         <collision>
             <geometry>
-                <sphere radius="0.05"/>
+                <sphere radius="0.08"/>
             </geometry>
         </collision>
-        <xacro:inertial_cylinder mass="0.1" length="0.04" radius="0.05">
+        <xacro:inertial_cylinder mass="0.1" length="0.04" radius="0.08">
             <origin xyz="0 0 0" rpy="0 0 0"/>
         </xacro:inertial_cylinder>
@@ -93,5 +93,5 @@
         <visual>
             <geometry>
-                <sphere radius="0.05"/>
+                <sphere radius="0.08"/>
             </geometry>
             <material name="black"/>
@@ -99,8 +99,8 @@
         <collision>
             <geometry>
-                <sphere radius="0.05"/>
+                <sphere radius="0.08"/>
             </geometry>
         </collision>
-        <xacro:inertial_sphere mass="0.1" radius="0.05">
+        <xacro:inertial_sphere mass="0.1" radius="0.08">
             <origin xyz="0 0 0" rpy="0 0 0"/>
         </xacro:inertial_sphere>

Commit message: Create footprint link

File: sd_simulation/description/body.xacro (robot description, xacro)
@@ -3,4 +3,11 @@
     <!-- BASE LINK -->
     <link name="base_link"/>
+    <!-- BASE FOOTPRINT LINK -->
+    <joint name="base_footprint_joint" type="fixed">
+        <parent link="base_link"/>
+        <child link="base_footprint"/>
+        <origin xyz="0 0 0"/>
+    </joint>
+    <link name="base_footprint"/>
     <!-- CHASSIS LINK -->
     <joint name="chassis_joint" type="fixed">

Commit message: Change body shape and caster wheel geometry

File: sd_simulation/description/body.xacro (robot description, xacro)
@@ -14,11 +14,11 @@
         <parent link="base_link"/>
         <child link="chassis"/>
-        <origin xyz="-0.1 0 0"/>
+        <origin xyz="0 0 0.075"/>
     </joint>
     <link name="chassis">
         <visual>
-            <origin xyz="0.15 0 0.075"/>
+            <origin xyz="0 0 0"/>
             <geometry>
-                <box size="0.3 0.3 0.15"/>
+                <box size="0.4 0.2 0.15"/>
             </geometry>
             <!-- Color for RVIZ -->
@@ -26,11 +26,11 @@
         </visual>
         <collision>
-            <origin xyz="0.15 0 0.075"/>
+            <origin xyz="0 0 0"/>
             <geometry>
-                <box size="0.3 0.3 0.15"/>
+                <box size="0.4 0.2 0.15"/>
             </geometry>
         </collision>
-        <xacro:inertial_box mass="0.5" x="0.3" y="0.3" z="0.15">
-            <origin xyz="0.15 0 0.075" rpy="0 0 0"/>
+        <xacro:inertial_box mass="0.5" x="0.4" y="0.2" z="0.15">
+            <origin xyz="0 0 0" rpy="0 0 0"/>
         </xacro:inertial_box>
     </link>
@@ -43,5 +43,5 @@
         <parent link="base_link"/>
         <child link="left_wheel"/>
-        <origin xyz="0 0.175 0" rpy="-${pi/2} 0 0" />
+        <origin xyz="-0.1 0.125 0" rpy="-${pi/2} 0 0"/>
         <axis xyz="0 0 1"/>
     </joint>
@@ -69,5 +69,5 @@
         <parent link="base_link"/>
         <child link="right_wheel"/>
-        <origin xyz="0 -0.175 0" rpy="${pi/2} 0 0" />
+        <origin xyz="-0.1 -0.125 0" rpy="${pi/2} 0 0"/>
         <axis xyz="0 0 -1"/>
     </joint>
@@ -93,26 +93,26 @@
     <!-- CASTER WHEEL LINK -->
     <joint name="caster_wheel_joint" type="fixed">
-        <parent link="chassis"/>
+        <parent link="base_link"/>
         <child link="caster_wheel"/>
-        <origin xyz="0.24 0 0"/>
+        <origin xyz="0.14 0 -0.04" rpy="-${pi/2} 0 0"/>
     </joint>
     <link name="caster_wheel">
         <visual>
             <geometry>
-                <sphere radius="0.08"/>
+                <cylinder radius="0.04" length="0.04"/>
             </geometry>
-            <material name="black"/>
+            <material name="yellow"/>
         </visual>
         <collision>
             <geometry>
-                <sphere radius="0.08"/>
+                <sphere radius="0.04"/>
             </geometry>
         </collision>
-        <xacro:inertial_sphere mass="0.1" radius="0.08">
+        <xacro:inertial_cylinder mass="0.1" length="0.04" radius="0.04">
             <origin xyz="0 0 0" rpy="0 0 0"/>
-        </xacro:inertial_sphere>
+        </xacro:inertial_cylinder>
     </link>
     <gazebo reference="caster_wheel">
-        <material>Gazebo/Black</material>
+        <material>Gazebo/Wood</material>
         <mu1 value="0.001"/>
         <mu2 value="0.001"/>

Commit message: Convert to skid steer drive

File: sd_simulation/description/body.xacro (robot description, xacro)
@@ -39,12 +39,12 @@
         <material>Gazebo/White</material>
     </gazebo>
-    <!-- LEFT WHEEL LINK -->
-    <joint name="left_wheel_joint" type="continuous">
+    <!-- FRONT LEFT WHEEL LINK -->
+    <joint name="front_left_wheel_joint" type="continuous">
         <parent link="base_link"/>
-        <child link="left_wheel"/>
-        <origin xyz="-0.1 0.125 0" rpy="-${pi/2} 0 0"/>
+        <child link="front_left_wheel"/>
+        <origin xyz="0.1 0.125 0" rpy="-${pi/2} 0 0"/>
         <axis xyz="0 0 1"/>
     </joint>
-    <link name="left_wheel">
+    <link name="front_left_wheel">
         <visual>
             <geometry>
@@ -62,15 +62,15 @@
         </xacro:inertial_cylinder>
     </link>
-    <gazebo reference="left_wheel">
+    <gazebo reference="front_left_wheel">
         <material>Gazebo/Wood</material>
     </gazebo>
-    <!-- RIGHT WHEEL LINK -->
-    <joint name="right_wheel_joint" type="continuous">
+    <!-- FRONT RIGHT WHEEL LINK -->
+    <joint name="front_right_wheel_joint" type="continuous">
         <parent link="base_link"/>
-        <child link="right_wheel"/>
-        <origin xyz="-0.1 -0.125 0" rpy="${pi/2} 0 0"/>
+        <child link="front_right_wheel"/>
+        <origin xyz="0.1 -0.125 0" rpy="${pi/2} 0 0"/>
         <axis xyz="0 0 -1"/>
     </joint>
-    <link name="right_wheel">
+    <link name="front_right_wheel">
         <visual>
             <geometry>
@@ -88,17 +88,18 @@
         </xacro:inertial_cylinder>
     </link>
-    <gazebo reference="right_wheel">
+    <gazebo reference="front_right_wheel">
         <material>Gazebo/Wood</material>
     </gazebo>
-    <!-- CASTER WHEEL LINK -->
-    <joint name="caster_wheel_joint" type="fixed">
+    <!-- BACK LEFT WHEEL LINK -->
+    <joint name="back_left_wheel_joint" type="continuous">
         <parent link="base_link"/>
-        <child link="caster_wheel"/>
-        <origin xyz="0.14 0 -0.04" rpy="-${pi/2} 0 0"/>
+        <child link="back_left_wheel"/>
+        <origin xyz="-0.1 0.125 0" rpy="-${pi/2} 0 0"/>
+        <axis xyz="0 0 1"/>
     </joint>
-    <link name="caster_wheel">
+    <link name="back_left_wheel">
         <visual>
             <geometry>
-                <cylinder radius="0.04" length="0.04"/>
+                <cylinder radius="0.08" length="0.04"/>
             </geometry>
             <material name="yellow"/>
@@ -106,15 +107,39 @@
         <collision>
             <geometry>
-                <sphere radius="0.04"/>
+                <sphere radius="0.08"/>
             </geometry>
         </collision>
-        <xacro:inertial_cylinder mass="0.1" length="0.04" radius="0.04">
+        <xacro:inertial_cylinder mass="0.1" length="0.04" radius="0.08">
             <origin xyz="0 0 0" rpy="0 0 0"/>
         </xacro:inertial_cylinder>
     </link>
-    <gazebo reference="caster_wheel">
+    <gazebo reference="back_left_wheel">
         <material>Gazebo/Wood</material>
-        <mu1 value="0.001"/>
-        <mu2 value="0.001"/>
+    </gazebo>
+    <!-- BACK RIGHT WHEEL LINK -->
+    <joint name="back_right_wheel_joint" type="continuous">
+        <parent link="base_link"/>
+        <child link="back_right_wheel"/>
+        <origin xyz="-0.1 -0.125 0" rpy="${pi/2} 0 0"/>
+        <axis xyz="0 0 -1"/>
+    </joint>
+    <link name="back_right_wheel">
+        <visual>
+            <geometry>
+                <cylinder radius="0.08" length="0.04"/>
+            </geometry>
+            <material name="yellow"/>
+        </visual>
+        <collision>
+            <geometry>
+                <sphere radius="0.08"/>
+            </geometry>
+        </collision>
+        <xacro:inertial_cylinder mass="0.1" length="0.04" radius="0.08">
+            <origin xyz="0 0 0" rpy="0 0 0"/>
+        </xacro:inertial_cylinder>
+    </link>
+    <gazebo reference="back_right_wheel">
+        <material>Gazebo/Wood</material>
     </gazebo>
 </robot>

File: sd_simulation/description/gazebo_control.xacro (robot description, xacro)
@@ -2,30 +2,21 @@
 <robot xmlns:xacro="http://www.ros.org/wiki/xacro">
     <gazebo>
-        <plugin name='diff_drive' filename='libgazebo_ros_diff_drive.so'>
-            <!-- Wheel Information -->
-            <leftJoint>left_wheel_joint</leftJoint>
-            <rightJoint>right_wheel_joint</rightJoint>
+        <plugin name="skid_steer_drive_controller" filename="libgazebo_ros_skid_steer_drive.so">
+            <updateRate>100.0</updateRate>
+            <leftFrontJoint>front_left_wheel_joint</leftFrontJoint>
+            <rightFrontJoint>front_right_wheel_joint</rightFrontJoint>
+            <leftRearJoint>back_left_wheel_joint</leftRearJoint>
+            <rightRearJoint>back_right_wheel_joint</rightRearJoint>
             <wheelSeparation>0.25</wheelSeparation>
             <wheelDiameter>0.08</wheelDiameter>
-            <!-- Limits -->
-            <maxWheelTorque>200</maxWheelTorque>
-            <maxWheelAcceleration>10.0</maxWheelAcceleration>
-            <!-- Topics -->
+            <robotBaseFrame>base_link</robotBaseFrame>
+            <torque>20</torque>
+            <broadcastTF>true</broadcastTF>
             <commandTopic>cmd_vel</commandTopic>
             <odometryTopic>odom</odometryTopic>
-            <!-- Output -->
             <odometryFrame>odom</odometryFrame>
-            <robotBaseFrame>base_link</robotBaseFrame>
-            <!-- Others -->
-            <rosDebugLevel>Debug</rosDebugLevel>
-            <publishTf>true</publishTf>
-            <publishWheelTF>false</publishWheelTF>
-            <publishOdom>true</publishOdom>
-            <publishOdomTF>true</publishOdomTF>
-            <publishWheelJointState>true</publishWheelJointState>
-            <wheelAcceleration>1.8</wheelAcceleration>
-            <wheelTorque>5</wheelTorque>
-            <updateRate>100</updateRate>
-            <odometrySource>world</odometrySource>
+            <covariance_x>0.0001</covariance_x>
+            <covariance_y>0.0001</covariance_y>
+            <covariance_yaw>0.01</covariance_yaw>
         </plugin>
     </gazebo>

Commit message: Make base_footprint parent of base_link

File: sd_simulation/description/body.xacro (robot description, xacro)
@@ -5,6 +5,6 @@
     <!-- BASE FOOTPRINT LINK -->
     <joint name="base_footprint_joint" type="fixed">
-        <parent link="base_link"/>
-        <child link="base_footprint"/>
+        <parent link="base_footprint"/>
+        <child link="base_link"/>
         <origin xyz="0 0 0"/>
     </joint>

File: sd_simulation/description/gazebo_control.xacro (robot description, xacro)
@@ -10,5 +10,5 @@
             <wheelSeparation>0.25</wheelSeparation>
             <wheelDiameter>0.08</wheelDiameter>
-            <robotBaseFrame>base_link</robotBaseFrame>
+            <robotBaseFrame>base_footprint</robotBaseFrame>
             <torque>20</torque>
             <broadcastTF>true</broadcastTF>
