Commit message: Fix Lidar parent to chassis

File: sd_simulation/description/lidar.xacro (robot description, xacro)
@@ -2,5 +2,5 @@
 <robot xmlns:xacro="http://www.ros.org/wiki/xacro" >
     <joint name="laser_joint" type="fixed">
-        <parent link="base_link"/>
+        <parent link="chassis"/>
         <child link="laser_frame"/>
         <origin xyz="0.1 0 0.175" rpy="0 0 0"/>

Commit message: Use custom Lidar

File: sd_simulation/description/lidar.xacro (robot description, xacro)
@@ -1,13 +1,13 @@
 <?xml version="1.0"?>
 <robot xmlns:xacro="http://www.ros.org/wiki/xacro" >
-    <joint name="laser_joint" type="fixed">
+    <joint name="head_lidar_joint" type="fixed">
         <parent link="base_link"/>
-        <child link="laser_frame"/>
-        <origin xyz="0.1 0 0.175" rpy="0 0 0"/>
+        <child link="head_lidar"/>
+        <origin xyz="0 0 0.2" rpy="0 0 0"/>
     </joint>
-    <link name="laser_frame">
+    <link name="head_lidar">
         <visual>
             <geometry>
-                <cylinder radius="0.05" length="0.04"/>
+                <cylinder radius="0.05" length="0.02"/>
             </geometry>
             <material name="red"/>
@@ -15,33 +15,43 @@
         <collision>
             <geometry>
-                <cylinder radius="0.05" length="0.04"/>
+                <cylinder radius="0.05" length="0.02"/>
             </geometry>
         </collision>
+        <xacro:inertial_cylinder mass="0.01" length="0.02" radius="0.05">
+            <origin xyz="0 0 0" rpy="0 0 0"/>
+        </xacro:inertial_cylinder>
     </link>
-    <gazebo reference="laser_frame">
+    <gazebo reference="head_lidar">
         <material>Gazebo/Red</material>
-        <sensor name="laser" type="ray">
+        <sensor name="head_lidar_sensor" type="ray">
             <pose> 0 0 0 0 0 0 </pose>
             <visualize>true</visualize>
-            <update_rate>10</update_rate>
+            <update_rate>40</update_rate>
             <ray>
                 <scan>
                     <horizontal>
-                        <samples>360</samples>
-                        <min_angle>-3.14</min_angle>
-                        <max_angle>3.14</max_angle>
+                        <samples>720</samples>
+                        <resolution>1</resolution>
+                        <min_angle>-3.141</min_angle>
+                        <max_angle>3.141</max_angle>
                     </horizontal>
                 </scan>
                 <range>
-                    <min>0.3</min>
-                    <max>12</max>
+                    <min>0.1</min>
+                    <max>10.0</max>
                 </range>
             </ray>
-            <plugin name="laser_controller" filename="libgazebo_ros_ray_sensor.so">
-                <ros>
-                    <argument>~/out:=scan</argument>
-                </ros>
-                <output_type>sensor_msgs/LaserScan</output_type>
-                <frame_name>laser_frame</frame_name>
+            <noise>
+                <type>gaussian</type>
+                <!-- Noise parameters based on published spec for Hokuyo laser
+                    achieving "+-30mm" accuracy at range < 10m.  A mean of 0.0m and
+                    stddev of 0.01m will put 99.7% of samples within 0.03m of the true
+                    reading. -->
+                <mean>0.0</mean>
+                <stddev>0.01</stddev>
+            </noise>
+            <plugin name="laser_controller" filename="libgazebo_ros_laser.so">
+                <topicName>/soonduck/lidar/scan</topicName>
+                <frameName>head_lidar</frameName>
             </plugin>
         </sensor>

File: sd_simulation/description/soonduck.xacro (robot description, xacro)
@@ -4,9 +4,10 @@
     <xacro:include filename="colors.xacro" />
     <xacro:include filename="body.xacro" />
-    <xacro:include filename="$(find gazebo_plugins)/test/multi_robot_scenario/xacro/laser/hokuyo.xacro" />
+    <!-- Example Hokuyo Lidar -->
+    <!-- <xacro:include filename="$(find gazebo_plugins)/test/multi_robot_scenario/xacro/laser/hokuyo.xacro" />
     <xacro:laser name="lidar" parent="base_link"
         xyz="0 0 0.2" rpy="0 0 0"
-        meshes="package://gazebo_plugins/test/multi_robot_scenario/meshes/laser" />
-    <!-- <xacro:include filename="lidar.xacro"/> -->
+        meshes="package://gazebo_plugins/test/multi_robot_scenario/meshes/laser" /> -->
+    <xacro:include filename="lidar.xacro"/>
     <xacro:include filename="camera.xacro"/>
     <!-- <xacro:if value="$(arg use_ros2_control)">
